Commit message: Rename optical frame links for consistency in URDF and RViz configuration

File: urdf/zed_macro.urdf.xacro (robot description, xacro)
@@ -191,9 +191,9 @@
         <origin xyz="${optical_offset_x} ${baseline/2} 0" rpy="0 0 0" />
       </joint>
-      <link name="${name}_left_camera_optical_frame"/>
+<link name="${name}_left_camera_frame_optical"/>
       <joint name="${name}_left_camera_optical_joint" type="fixed">
         <origin xyz="0 0 0" rpy="-${M_PI/2} 0.0 -${M_PI/2}"/>
         <parent link="${name}_left_camera_frame"/>
-        <child link="${name}_left_camera_optical_frame"/>
+<child link="${name}_left_camera_frame_optical"/>
       </joint>
       <!-- Right Camera -->
@@ -220,9 +220,9 @@
         <origin xyz="${optical_offset_x} -${baseline/2} 0" rpy="0 0 0" />
       </joint>
-      <link name="${name}_right_camera_optical_frame"/>
+<link name="${name}_right_camera_frame_optical"/>
       <joint name="${name}_right_camera_optical_joint" type="fixed">
         <origin xyz="0 0 0" rpy="-${M_PI/2} 0.0 -${M_PI/2}"/>
         <parent link="${name}_right_camera_frame"/>
-        <child link="${name}_right_camera_optical_frame"/>
+<child link="${name}_right_camera_frame_optical"/>
       </joint>
       <!-- ZED2 Sensors -->
@@ -262,9 +262,9 @@
         <origin xyz="${optical_offset_x} 0 0" rpy="0 0 0" />
       </joint>
-      <link name="${name}_camera_optical_frame"/>
+<link name="${name}_camera_frame_optical"/>
       <joint name="${name}_camera_optical_joint" type="fixed">
         <origin xyz="0 0 0" rpy="-${M_PI/2} 0.0 -${M_PI/2}"/>
         <parent link="${name}_camera_frame"/>
-        <child link="${name}_camera_optical_frame"/>
+<child link="${name}_camera_frame_optical"/>
       </joint>
     </xacro:if>

Commit message: fix: cleanup whitespace

File: urdf/zed_macro.urdf.xacro (robot description, xacro)
@@ -17,5 +17,5 @@
 <robot xmlns:xacro="http://wiki.ros.org/xacro">
   <xacro:include filename="package://zed_description/urdf/include/materials.urdf.xacro" />
-  <xacro:property name="M_PI"     value="3.1415926535897931" />
+  <xacro:property name="M_PI" value="3.1415926535897931" />
   <!--
     Parameters:
@@ -191,9 +191,9 @@
         <origin xyz="${optical_offset_x} ${baseline/2} 0" rpy="0 0 0" />
       </joint>
-<link name="${name}_left_camera_frame_optical"/>
+      <link name="${name}_left_camera_frame_optical"/>
       <joint name="${name}_left_camera_optical_joint" type="fixed">
         <origin xyz="0 0 0" rpy="-${M_PI/2} 0.0 -${M_PI/2}"/>
         <parent link="${name}_left_camera_frame"/>
-<child link="${name}_left_camera_frame_optical"/>
+        <child link="${name}_left_camera_frame_optical"/>
       </joint>
       <!-- Right Camera -->
@@ -220,9 +220,9 @@
         <origin xyz="${optical_offset_x} -${baseline/2} 0" rpy="0 0 0" />
       </joint>
-<link name="${name}_right_camera_frame_optical"/>
+      <link name="${name}_right_camera_frame_optical"/>
       <joint name="${name}_right_camera_optical_joint" type="fixed">
         <origin xyz="0 0 0" rpy="-${M_PI/2} 0.0 -${M_PI/2}"/>
         <parent link="${name}_right_camera_frame"/>
-<child link="${name}_right_camera_frame_optical"/>
+        <child link="${name}_right_camera_frame_optical"/>
       </joint>
       <!-- ZED2 Sensors -->
@@ -262,9 +262,9 @@
         <origin xyz="${optical_offset_x} 0 0" rpy="0 0 0" />
       </joint>
-<link name="${name}_camera_frame_optical"/>
+      <link name="${name}_camera_frame_optical"/>
       <joint name="${name}_camera_optical_joint" type="fixed">
         <origin xyz="0 0 0" rpy="-${M_PI/2} 0.0 -${M_PI/2}"/>
         <parent link="${name}_camera_frame"/>
-<child link="${name}_camera_frame_optical"/>
+        <child link="${name}_camera_frame_optical"/>
       </joint>
     </xacro:if>
